File: hw/m68kcomp2.kicad_sch (KiCad schematic)
At the start: 38 parts, among them J1 SWRST, SW1 SWRST, U1 GAL20V8, U10 mc68881, U11 74HC393, U2 GAL16V8, U3 NE555D, U4 74HC10, U5 74LS14, U6 74HC148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

Commit message: finished the footprints
Parts:
- SW1: footprint (none) -> Button_Switch_SMD:SW_SPST_EVPBF
Changed lines of the file:
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@@
     (property "Reference" "SW1" (id 0) (at 19.05 130.81 0))
     (property "Value" "SWRST" (id 1) (at 19.05 138.43 0))
-    (property "Footprint" "" (id 2) (at 19.05 130.81 0)
+    (property "Footprint" "Button_Switch_SMD:SW_SPST_EVPBF" (id 2) (at 19.05 130.81 0)
       (effects (font (size 1.27 1.27)) hide)
     )
@@
     )
     (path "/bb1f193c-4db0-43b5-9bb8-e99d45af99a9/f31c27a3-c4bf-40dc-b93d-16593509c4e7"
-      (reference "C8") (unit 1) (value "10uF") (footprint "")
+      (reference "C8") (unit 1) (value "10uF") (footprint "Capacitor_SMD:CP_Elec_4x4.5")
     )
     (path "/bb1f193c-4db0-43b5-9bb8-e99d45af99a9/0fb7fc9c-fcf7-47c1-988f-7294d0311d51"
-      (reference "C9") (unit 1) (value "22uF") (footprint "")
+      (reference "C9") (unit 1) (value "22uF") (footprint "Capacitor_SMD:CP_Elec_4x4.5")
     )
     (path "/bb1f193c-4db0-43b5-9bb8-e99d45af99a9/15000b20-85db-448a-b844-c0aa86bc87ce"
@@
     )
     (path "/d7997dcc-7f79-4011-8eff-8d684ebed9c8"
-      (reference "SW1") (unit 1) (value "SWRST") (footprint "")
+      (reference "SW1") (unit 1) (value "SWRST") (footprint "Button_Switch_SMD:SW_SPST_EVPBF")
     )
     (path "/bb1f193c-4db0-43b5-9bb8-e99d45af99a9/212d34c3-ef9b-43fe-be7e-785b087f50df"
@@
     )
     (path "/018b57af-ff7d-4307-85ac-81c5bb9e22f2/5569c6f5-5fd7-49d3-b3ab-5c5234315d6a"
-      (reference "U15") (unit 1) (value "mouse") (footprint "")
+      (reference "U15") (unit 1) (value "mouse") (footprint "m68kcomp2:minidin6")
     )
     (path "/018b57af-ff7d-4307-85ac-81c5bb9e22f2/900bd744-39ea-4eca-848c-3ba10fa82615"
-      (reference "U16") (unit 1) (value "kbd") (footprint "")
+      (reference "U16") (unit 1) (value "kbd") (footprint "m68kcomp2:minidin6")
     )
     (path "/018b57af-ff7d-4307-85ac-81c5bb9e22f2/8ab334f6-0907-4b4c-9e7b-262500583ec9"
@@
     )
     (path "/018b57af-ff7d-4307-85ac-81c5bb9e22f2/4e6f63e0-aae7-448c-af4d-a1af0761168e"
-      (reference "U23") (unit 1) (value "sdcard") (footprint "")
+      (reference "U23") (unit 1) (value "sdcard") (footprint "Connector_Card:SD_TE_2041021")
     )
     (path "/018b57af-ff7d-4307-85ac-81c5bb9e22f2/c8079437-ca81-45a2-920d-9158027f50d7"

Commit message: fixed resistor footprint assignments, changed PCB to 4-layer
Parts:
- R3, R4: footprint OptoDevice:R_LDR_D13.8mm_P9.0mm_Vertical -> Resistor_SMD:R_0805_2012Metric_Pad1.20x1.40mm_HandSolder
Changed lines of the file:
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@@
       (effects (font (size 1.27 1.27)) (justify left))
     )
-    (property "Footprint" "OptoDevice:R_LDR_D13.8mm_P9.0mm_Vertical" (id 2) (at 77.47 154.178 90)
+    (property "Footprint" "Resistor_SMD:R_0805_2012Metric_Pad1.20x1.40mm_HandSolder" (id 2) (at 77.47 154.178 90)
       (effects (font (size 1.27 1.27)) hide)
     )
@@
       (effects (font (size 1.27 1.27)) (justify left))
     )
-    (property "Footprint" "OptoDevice:R_LDR_D13.8mm_P9.0mm_Vertical" (id 2) (at 139.192 191.77 90)
+    (property "Footprint" "Resistor_SMD:R_0805_2012Metric_Pad1.20x1.40mm_HandSolder" (id 2) (at 139.192 191.77 90)
       (effects (font (size 1.27 1.27)) hide)
     )
@@
     )
     (path "/9508d616-40da-4229-8e75-ddcf500da2cc"
-      (reference "R3") (unit 1) (value "4k7") (footprint "OptoDevice:R_LDR_D13.8mm_P9.0mm_Vertical")
+      (reference "R3") (unit 1) (value "4k7") (footprint "Resistor_SMD:R_0805_2012Metric_Pad1.20x1.40mm_HandSolder")
     )
     (path "/b99cfdd4-1443-4e14-9c8b-a346be8294ac"
-      (reference "R4") (unit 1) (value "4k7") (footprint "OptoDevice:R_LDR_D13.8mm_P9.0mm_Vertical")
+      (reference "R4") (unit 1) (value "4k7") (footprint "Resistor_SMD:R_0805_2012Metric_Pad1.20x1.40mm_HandSolder")
     )
     (path "/018b57af-ff7d-4307-85ac-81c5bb9e22f2/529b1525-6dc5-4706-a288-e328b5ead0a5"
-      (reference "R5") (unit 1) (value "4k7") (footprint "OptoDevice:R_LDR_D13.8mm_P9.0mm_Vertical")
+      (reference "R5") (unit 1) (value "4k7") (footprint "Resistor_SMD:R_0805_2012Metric_Pad1.20x1.40mm_HandSolder")
     )
     (path "/018b57af-ff7d-4307-85ac-81c5bb9e22f2/af7f1839-d4ec-4fbe-a95d-d9f8132fda16"
-      (reference "R6") (unit 1) (value "1k") (footprint "OptoDevice:R_LDR_D13.8mm_P9.0mm_Vertical")
+      (reference "R6") (unit 1) (value "1k") (footprint "Resistor_SMD:R_0805_2012Metric_Pad1.20x1.40mm_HandSolder")
     )
     (path "/018b57af-ff7d-4307-85ac-81c5bb9e22f2/e3880d25-af4b-47d7-a246-101205e47723"
-      (reference "R7") (unit 1) (value "1k") (footprint "OptoDevice:R_LDR_D13.8mm_P9.0mm_Vertical")
+      (reference "R7") (unit 1) (value "1k") (footprint "Resistor_SMD:R_0805_2012Metric_Pad1.20x1.40mm_HandSolder")
     )
     (path "/3086e7bb-ee82-4de0-9e96-a315fb5211a4"

Commit message: 32bit buses take a lot of space
Parts:
- added TP13: TPDS, TestPoint:TestPoint_Pad_D1.5mm, symbol Connector:TestPoint_Probe
Connections:
- net ~{DS}: now also U8.K2 (~{DS}), TP13.1
- no-connect marks 35 -> 34
Other:
- moved on the sheet: D2, D3, D4
